File: gfx-9918.kicad_pcb (KiCad board)
At the start: 2 copper layers, 50 x 150 mm, 28 parts, among them J1 GFX_Connector_Input, J2 RCA_Conn, J3 RCA_Conn, J4 RCA_Conn, U1 TMS9918, U2 74HCT04, U3 74HCT574, U4 74HCT574, U5 74HCT574, U6 62256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

Commit message: Update to latest libs to use power connectors in first part for multipart symbols
Connections:
- net /Input connector & power/A0 renamed /Card connector & power/A0
- net /Input connector & power/BUSDIR renamed /Card connector & power/BUSDIR
- net /Input connector & power/DATA0 renamed /Card connector & power/DATA0
- net /Input connector & power/DATA1 renamed /Card connector & power/DATA1
- net /Input connector & power/DATA2 renamed /Card connector & power/DATA2
- net /Input connector & power/DATA3 renamed /Card connector & power/DATA3
- net /Input connector & power/DATA4 renamed /Card connector & power/DATA4
- net /Input connector & power/DATA5 renamed /Card connector & power/DATA5
- net /Input connector & power/DATA6 renamed /Card connector & power/DATA6
- net /Input connector & power/DATA7 renamed /Card connector & power/DATA7
- net /Input connector & power/SOUNDOUT renamed /Card connector & power/SOUNDOUT
- net /Input connector & power/~INT renamed /Card connector & power/~INT
- net /Input connector & power/~RD renamed /Card connector & power/~RD
- net /Input connector & power/~RESET renamed /Card connector & power/~RESET
- net /Input connector & power/~VDPIOSL renamed /Card connector & power/~VDPIOSL
- net /Input connector & power/~WR renamed /Card connector & power/~WR

Commit message: Upgrade project files to KiCad 6
Connections:
- net /Card connector & power/~INT renamed /Card connector & power/~{INT}
- net /Card connector & power/~RD renamed /Card connector & power/~{RD}
- net /Card connector & power/~RESET renamed /Card connector & power/~{RESET}
- net /Card connector & power/~VDPIOSL renamed /Card connector & power/~{VDPIOSL}
- net /Card connector & power/~WR renamed /Card connector & power/~{WR}
- net /Interface Decoding Logic/~CSW renamed /Interface Decoding Logic/~{CSW}
- net /VRAM Decoding Logic/~CAS renamed /VRAM Decoding Logic/~{CAS}
- net /VRAM Decoding Logic/~RAS renamed /VRAM Decoding Logic/~{RAS}
- net /VRAM Decoding Logic/~WR renamed /VRAM Decoding Logic/~{WR}
Other:
- net class Default removed
- net class Power removed
